File: pcb/stm32-tf.brd (EAGLE design)
At the start: 6.9 x 6.9 mm, 79 parts, among them IC1 FT232RL, Q1 8mhz, Q2 32khz, Q3 IRF530, Q4 IRF530, U1 STM32F10XRXT6

Commit message: estimasi harga
Parts:
- C-USER1, C-USER2: value 10nf -> 100nf
Changed lines of the file:
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@@
 <element name="R-USER1" library="resistor" package="R1206" value="4k7" x="83.312" y="44.45" rot="MR0"/>
 <element name="C-RST" library="resistor" package="C1206" value="100nf" x="53.467" y="33.909" rot="MR180"/>
-<element name="C-USER1" library="resistor" package="C1206" value="10nf" x="83.312" y="42.291" rot="MR180"/>
+<element name="C-USER1" library="resistor" package="C1206" value="100nf" x="83.312" y="42.291" rot="MR180"/>
 <element name="USER2" library="switch-omron" package="B3F-10XX" value="" x="93.091" y="50.546" rot="R90">
 <attribute name="OC_NEWARK" value="36M3542" x="82.042" y="39.878" size="1.778" layer="27" rot="R90" display="off"/>
@@
 </element>
 <element name="R-USER2" library="resistor" package="R1206" value="4k7" x="92.202" y="42.164" rot="MR0"/>
-<element name="C-USER2" library="resistor" package="C1206" value="10nf" x="92.202" y="44.323" rot="MR180"/>
+<element name="C-USER2" library="resistor" package="C1206" value="100nf" x="92.202" y="44.323" rot="MR180"/>
 <element name="JPUSER" library="pinhead" package="1X02" value="" x="87.503" y="38.862"/>
 <element name="OK1" library="optocoupler" package="DIL06" value="H11L1M" x="74.041" y="31.115">
