File: pcb/stm32-tf.sch (EAGLE design)
At the start: 79 parts, among them IC1 FT232RL, Q1 8mhz, Q2 32khz, Q3 IRF530, Q4 IRF530, U1 STM32F10XRXT6

Commit message: estimasi harga
Parts:
- C-USER1, C-USER2: value 10nf -> 100nf
Changed lines of the file:
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@@
 <part name="R-USER1" library="resistor" deviceset="R-EU_" device="R1206" value="4k7"/>
 <part name="C-RST" library="resistor" deviceset="C-EU" device="C1206" value="100nf"/>
-<part name="C-USER1" library="resistor" deviceset="C-EU" device="C1206" value="10nf"/>
+<part name="C-USER1" library="resistor" deviceset="C-EU" device="C1206" value="100nf"/>
 <part name="USER2" library="switch-omron" deviceset="10-XX" device=""/>
 <part name="R-USER2" library="resistor" deviceset="R-EU_" device="R1206" value="4k7"/>
-<part name="C-USER2" library="resistor" deviceset="C-EU" device="C1206" value="10nf"/>
+<part name="C-USER2" library="resistor" deviceset="C-EU" device="C1206" value="100nf"/>
 <part name="JPUSER" library="pinhead" deviceset="PINHD-1X2" device=""/>
 <part name="OK1" library="optocoupler" deviceset="H11L*M" device="" technology="1"/>
